File: hardware/ThermistorHub/ThermistorHub/untitled.kicad_sch (KiCad schematic)
At the start: 1 part, among them J110 Micro_SD_Card_Det_Hirose_DM3AT

Commit message: 発注
Parts:
- added C107: 10uF, Capacitor_THT:C_Axial_L3.8mm_D2.6mm_P7.50mm_Horizontal, symbol Device:C
- added C108: 0.1uF, Capacitor_THT:C_Axial_L3.8mm_D2.6mm_P7.50mm_Horizontal, symbol Device:C
- added R107, R108, R110, R111: 10k, Resistor_THT:R_Axial_DIN0204_L3.6mm_D1.6mm_P5.08mm_Horizontal, symbol Device:R
- added R109: 22Ω, Resistor_THT:R_Axial_DIN0204_L3.6mm_D1.6mm_P5.08mm_Horizontal, symbol Device:R
- J110: footprint (none) -> Connector_Card:microSD_HC_Hirose_DM3AT-SF-PEJM5
Connections:
- net DET_A is gone; now on net GND: J110.10 (DET_A)
- net VSS is gone; now on net GND: J110.6 (VSS)
- net CLK: now also R109.1; no longer J110.5 (CLK)
- net CMD: now also R108.2
- net GND: now also C107.1, C108.1
- net VDD: now also C107.2, C108.2, R107.1, R108.1, R110.1, R111.1
- net DAT1: no longer names the net of J110.8 (DAT1)
- net DAT1: now also R111.2
- net DAT2: no longer names the net of J110.1 (DAT2)
- net DAT2: now also R107.2
- net DAT3/CD: no longer names the net of J110.2 (DAT3/CD)
- net DAT3/CD: now also R110.2
- new net: J110.5 (CLK), R109.2
