File: hardware/ThermistorHub/ThermistorHub/SD.kicad_sch (KiCad schematic)
At the start: 8 parts, among them J110 Micro_SD_Card_Det_Hirose_DM3AT

Commit message: 諸々
Parts:
- added R306: 10k, Resistor_THT:R_Axial_DIN0204_L3.6mm_D1.6mm_P5.08mm_Horizontal, symbol Device:R
- renumbered C108 to C301, C107 to C302, J110 to J301, R108 to R301, R109 to R302, R111 to R303, R110 to R304, R107 to R305
Connections:
- net DAT0: now also R306.2
- net VDD: now also R306.1
Other:
- moved on the sheet: R301
Changed lines of the file:
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@@
+	)
+	(junction
+		(at 90.17 106.68)
+		(diameter 0)
+		(color 0 0 0 0)
+	)
+	(junction
+		(at 86.36 96.52)
+		(diameter 0)
+		(color 0 0 0 0)
 	)
 	(junction
@@
 	)
 	(junction
+		(at 86.36 85.09)
+		(diameter 0)
+		(color 0 0 0 0)
+	)
+	(junction
 		(at 118.11 69.85)
 		(diameter 0)
 		(color 0 0 0 0)
 	)
-	(junction
-		(at 90.17 96.52)
-		(diameter 0)
-		(color 0 0 0 0)
-	)
 	(no_connect
 		(at 135.89 114.3)
@@
 	(wire
 		(pts
+			(xy 90.17 93.98) (xy 90.17 106.68)
+		)
+		(stroke
+			(width 0)
+			(type default)
+		)
+	)
+	(wire
+		(pts
 			(xy 115.57 74.93) (xy 118.11 74.93)
 		)
@@
 	(wire
 		(pts
+			(xy 90.17 86.36) (xy 90.17 85.09)
+		)
+		(stroke
+			(width 0)
+			(type default)
+		)
+	)
+	(wire
+		(pts
 			(xy 105.41 74.93) (xy 105.41 88.9)
 		)
@@
 	(wire
 		(pts
-			(xy 90.17 83.82) (xy 90.17 86.36)
+			(xy 86.36 83.82) (xy 86.36 85.09)
 		)
 		(stroke
@@
 	(wire
 		(pts
-			(xy 90.17 93.98) (xy 90.17 96.52)
+			(xy 86.36 85.09) (xy 86.36 86.36)
+		)
+		(stroke
+			(width 0)
+			(type default)
+		)
+	)
+	(wire
+		(pts
+			(xy 86.36 93.98) (xy 86.36 96.52)
 		)
 		(stroke
@@
 	(wire
 		(pts
-			(xy 81.28 106.68) (xy 135.89 106.68)
+			(xy 81.28 106.68) (xy 90.17 106.68)
 		)
 		(stroke
@@
 	(wire
 		(pts
+			(xy 86.36 96.52) (xy 135.89 96.52)
+		)
+		(stroke
+			(width 0)
+			(type default)
+		)
+	)
+	(wire
+		(pts
 			(xy 81.28 101.6) (xy 92.71 101.6)
 		)
@@
 	(wire
 		(pts
-			(xy 81.28 96.52) (xy 90.17 96.52)
-		)
-		(stroke
-			(width 0)
-			(type default)
-		)
-	)
-	(wire
-		(pts
-			(xy 90.17 96.52) (xy 135.89 96.52)
+			(xy 90.17 106.68) (xy 135.89 106.68)
+		)
+		(stroke
+			(width 0)
+			(type default)
+		)
+	)
+	(wire
+		(pts
+			(xy 86.36 85.09) (xy 90.17 85.09)
+		)
+		(stroke
+			(width 0)
+			(type default)
+		)
+	)
+	(wire
+		(pts
+			(xy 81.28 96.52) (xy 86.36 96.52)
 		)
 		(stroke
@@
 		(dnp no)
 		(fields_autoplaced yes)
-		(property "Reference" "C107"
+		(property "Reference" "C302"
 			(at 111.76 81.28 90)
 			(effects
@@
 		)
 		(instances
-			(project ""
+			(project "ThermistorHub"
 				(path "/654b68be-bf39-4999-b2d7-5e3864aa249f/37f9d874-8f1a-4c45-8870-fefc55033c59"
-					(reference "C107")
+					(reference "C302")
 					(unit 1)
 				)
@@
 		(dnp no)
 		(fields_autoplaced yes)
-		(property "Reference" "#PWR0104"
+		(property "Reference" "#PWR0305"
 			(at 184.15 123.19 0)
 			(effects
@@
 		)
 		(instances
-			(project ""
+			(project "ThermistorHub"
 				(path "/654b68be-bf39-4999-b2d7-5e3864aa249f/37f9d874-8f1a-4c45-8870-fefc55033c59"
-					(reference "#PWR0104")
+					(reference "#PWR0305")
 					(unit 1)
 				)
@@
 	(symbol
 		(lib_id "power:VDD")
-		(at 90.17 83.82 0)
+		(at 86.36 83.82 0)
 		(unit 1)
 		(exclude_from_sim no)
@@
 		(dnp no)
 		(fields_autoplaced yes)
-		(property "Reference" "#PWR0107"
-			(at 90.17 87.63 0)
+		(property "Reference" "#PWR0301"
+			(at 86.36 87.63 0)
 			(effects
 				(font
@@
 		)
 		(property "Value" "VDD"
-			(at 90.17 78.74 0)
+			(at 86.36 78.74 0)
 			(effects
 				(font
@@
 		)
 		(property "Footprint" ""
-			(at 90.17 83.82 0)
+			(at 86.36 83.82 0)
 			(effects
 				(font
@@
 		)
 		(property "Datasheet" ""
-			(at 90.17 83.82 0)
+			(at 86.36 83.82 0)
 			(effects
 				(font
@@
 		)
 		(property "Description" "Power symbol creates a global label with name \"VDD\""
-			(at 90.17 83.82 0)
+			(at 86.36 83.82 0)
 			(effects
 				(font
@@
 		)
 		(instances
-			(project ""
+			(project "ThermistorHub"
 				(path "/654b68be-bf39-4999-b2d7-5e3864aa249f/37f9d874-8f1a-4c45-8870-fefc55033c59"
-					(reference "#PWR0107")
+					(reference "#PWR0301")
 					(unit 1)
 				)
@@
 		(on_board yes)
 		(dnp no)
-		(property "Reference" "R109"
+		(property "Reference" "R302"
 			(at 101.092 98.044 90)
 			(effects
@@
 		)
 		(instances
-			(project ""
+			(project "ThermistorHub"
 				(path "/654b68be-bf39-4999-b2d7-5e3864aa249f/37f9d874-8f1a-4c45-8870-fefc55033c59"
-					(reference "R109")
+					(reference "R302")
 					(unit 1)
 				)
@@
 		(dnp no)
 		(fields_autoplaced yes)
-		(property "Reference" "C108"
+		(property "Reference" "C301"
 			(at 111.76 67.31 90)
 			(effects
@@
 			(project "ThermistorHub"
 				(path "/654b68be-bf39-4999-b2d7-5e3864aa249f/37f9d874-8f1a-4c45-8870-fefc55033c59"
-					(reference "C108")
+					(reference "C301")
 					(unit 1)
 				)
@@
 		(dnp no)
 		(fields_autoplaced yes)
-		(property "Reference" "R111"
+		(property "Reference" "R303"
 			(at 127 78.7399 0)
 			(effects
@@
 			(project "ThermistorHub"
 				(path "/654b68be-bf39-4999-b2d7-5e3864aa249f/37f9d874-8f1a-4c45-8870-fefc55033c59"
-					(reference "R111")
+					(reference "R303")
 					(unit 1)
 				)
@@
 		(on_board yes)
 		(dnp no)
-		(property "Reference" "#PWR0106"
+		(property "Reference" "#PWR0302"
 			(at 105.41 96.52 0)
 			(effects
@@
 		)
 		(instances
-			(project ""
+			(project "ThermistorHub"
 				(path "/654b68be-bf39-4999-b2d7-5e3864aa249f/37f9d874-8f1a-4c45-8870-fefc55033c59"
-					(reference "#PWR0106")
+					(reference "#PWR0302")
 					(unit 1)
 				)
@@
 		(dnp no)
 		(fields_autoplaced yes)
-		(property "Reference" "J110"
+		(property "Reference" "J301"
 			(at 159.385 80.01 0)
 			(effects
@@
 		)
 		(instances
-			(project ""
+			(project "ThermistorHub"
 				(path "/654b68be-bf39-4999-b2d7-5e3864aa249f/37f9d874-8f1a-4c45-8870-fefc55033c59"
-					(reference "J110")
+					(reference "J301")
 					(unit 1)
 				)
@@
 		(on_board yes)
 		(dnp no)
-		(property "Reference" "R108"
-			(at 81.28 88.646 0)
+		(property "Reference" "R306"
+			(at 93.218 88.646 0)
 			(effects
 				(font
@@
 		)
 		(property "Value" "10k"
-			(at 81.28 91.186 0)
+			(at 93.472 91.44 0)
 			(effects
 				(font
@@
 		)
 		(instances
-			(project ""
+			(project "ThermistorHub"
 				(path "/654b68be-bf39-4999-b2d7-5e3864aa249f/37f9d874-8f1a-4c45-8870-fefc55033c59"
-					(reference "R108")
+					(reference "R306")
+					(unit 1)
+				)
+			)
+		)
+	)
+	(symbol
+		(lib_id "Device:R")
+		(at 86.36 90.17 0)
+		(unit 1)
+		(exclude_from_sim no)
+		(in_bom yes)
+		(on_board yes)
+		(dnp no)
+		(property "Reference" "R301"
+			(at 77.47 88.646 0)
+			(effects
+				(font
+					(size 1.27 1.27)
+				)
+				(justify left)
+			)
+		)
+		(property "Value" "10k"
+			(at 77.47 91.186 0)
+			(effects
+				(font
+					(size 1.27 1.27)
+				)
+				(justify left)
+			)
+		)
+		(property "Footprint" "Resistor_THT:R_Axial_DIN0204_L3.6mm_D1.6mm_P5.08mm_Horizontal"
+			(at 84.582 90.17 90)
+			(effects
+				(font
+					(size 1.27 1.27)
+				)
+				(hide yes)
+			)
+		)
+		(property "Datasheet" "~"
+			(at 86.36 90.17 0)
+			(effects
+				(font
+					(size 1.27 1.27)
+				)
+				(hide yes)
+			)
+		)
+		(property "Description" "Resistor"
+			(at 86.36 90.17 0)
+			(effects
+				(font
+					(size 1.27 1.27)
+				)
+				(hide yes)
+			)
+		)
+		(pin "1"
+		)
+		(pin "2"
+		)
+		(instances
+			(project "ThermistorHub"
+				(path "/654b68be-bf39-4999-b2d7-5e3864aa249f/37f9d874-8f1a-4c45-8870-fefc55033c59"
+					(reference "R301")
 					(unit 1)
 				)
@@
 		(dnp no)
 		(fields_autoplaced yes)
-		(property "Reference" "#PWR0108"
+		(property "Reference" "#PWR0304"
 			(at 118.11 118.11 0)
 			(effects
@@
 		)
 		(instances
-			(project ""
+			(project "ThermistorHub"
 				(path "/654b68be-bf39-4999-b2d7-5e3864aa249f/37f9d874-8f1a-4c45-8870-fefc55033c59"
-					(reference "#PWR0108")
+					(reference "#PWR0304")
 					(unit 1)
 				)
@@
 		(dnp no)
 		(fields_autoplaced yes)
-		(property "Reference" "R107"
+		(property "Reference" "R305"
 			(at 134.62 78.7399 0)
 			(effects
@@
 		)
 		(instances
-			(project ""
+			(project "ThermistorHub"
 				(path "/654b68be-bf39-4999-b2d7-5e3864aa249f/37f9d874-8f1a-4c45-8870-fefc55033c59"
-					(reference "R107")
+					(reference "R305")
 					(unit 1)
 				)
@@
 		(dnp no)
 		(fields_autoplaced yes)
-		(property "Reference" "#PWR0105"
+		(property "Reference" "#PWR0303"
 			(at 118.11 69.85 0)
 			(effects
@@
 		)
 		(instances
-			(project ""
+			(project "ThermistorHub"
 				(path "/654b68be-bf39-4999-b2d7-5e3864aa249f/37f9d874-8f1a-4c45-8870-fefc55033c59"
-					(reference "#PWR0105")
+					(reference "#PWR0303")
 					(unit 1)
 				)
@@
 		(dnp no)
 		(fields_autoplaced yes)
-		(property "Reference" "R110"
+		(property "Reference" "R304"
 			(at 130.81 78.7399 0)
 			(effects
@@
 			(project "ThermistorHub"
 				(path "/654b68be-bf39-4999-b2d7-5e3864aa249f/37f9d874-8f1a-4c45-8870-fefc55033c59"
-					(reference "R110")
+					(reference "R304")
 					(unit 1)
 				)
