File: hardware/ThermistorHub/ThermistorHub/Thermistor.kicad_sch (KiCad schematic)
At the start: 32 parts, among them J102 Thermistor1, J103 Thermistor5_BLK, J104 Thermistor2, J105 Thermistor5, J106 Thermistor3, J107 Thermistor6_BLK, J108 Thermistor6, J109 Thermistor4

Commit message: 発注
Parts:
- removed J103: Thermistor5_BLK, Connector_JST:JST_PH_B2B-PH-K_1x02_P2.00mm_Vertical, symbol Connector_Generic:Conn_01x02
- removed J107: Thermistor6_BLK, Connector_JST:JST_PH_B2B-PH-K_1x02_P2.00mm_Vertical, symbol Connector_Generic:Conn_01x02
- removed TP103, TP105, TP107, TP109, TP111: TestPoint, symbol Connector:TestPoint
- C101, C102, C103, C104, C105, C106: footprint Capacitor_SMD:C_0805_2012Metric -> Capacitor_THT:C_Axial_L3.8mm_D2.6mm_P7.50mm_Horizontal
- TP101, TP102, TP104, TP106, TP108, TP110, TP112: footprint (none) -> Connector_PinHeader_2.54mm:PinHeader_1x01_P2.54mm_Vertical
Other:
- moved on the sheet: TP106

Commit message: 諸々
Parts:
- renumbered C101 to C201, C102 to C202, C103 to C203, C104 to C204, C105 to C205, C106 to C206, J102 to J201, J104 to J202, J105 to J203, J106 to J204, J108 to J205, J109 to J206, R101 to R201, R102 to R202, R103 to R203, R104 to R204, R105 to R205, R106 to R206, TP101 to TP201, TP102 to TP202, TP104 to TP203, TP106 to TP204, TP108 to TP205, TP110 to TP206, TP112 to TP207
