File: hardware/ThermistorHub/ThermistorHub/ThermistorHub.kicad_pcb (KiCad board)
At the start: 2 copper layers, 80 x 50 mm, 46 parts, among them J101 Battery, J102 Thermistor1, J104 Thermistor2, J105 Thermistor5, J106 Thermistor3, J108 Thermistor6, J109 Thermistor4, J110 Micro_SD_Card_Det_Hirose_DM3AT, J111 GVCD, J112 GVDC

Commit message: 諸々
Parts:
- removed J112: GVDC, Connector_PinHeader_2.54mm:PinHeader_1x04_P2.54mm_Vertical
- added C401: 0.1uF, Capacitor_THT:C_Axial_L3.8mm_D2.6mm_P7.50mm_Horizontal, F.Cu at (107.4, 109.8)
- added J401: Conn_01x06, Connector_PinHeader_2.54mm:PinHeader_1x06_P2.54mm_Vertical, F.Cu at (103.9, 101.8)
- added ON: SW_SPDT, Button_Switch_THT:SW_Slide-03_Wuerth-WS-SLTV_10x2.5x6.4_P2.54mm, F.Cu at (137.1, 82.9)
- added R306: 10k, Resistor_THT:R_Axial_DIN0204_L3.6mm_D1.6mm_P5.08mm_Horizontal, F.Cu at (149.8, 90.6)
- moved R303 21.1 mm to (151.9, 90.6), turned to -90 degrees
- moved R301 18.1 mm to (154.0, 90.6), turned to -90 degrees
- moved R304 16.0 mm to (156.1, 90.6), turned to -90 degrees
- moved R305 15.1 mm to (158.2, 90.6), turned to -90 degrees
- moved J301 11.7 mm to (169.1, 96.5), turned to 90 degrees
- moved J101 10.3 mm to (145.6, 84.4)
- moved R302 9.57 mm to (136.5, 96.5)
- moved TP201 8.53 mm to (111.0, 126.0)
- moved R102 5.39 mm to (108.5, 120.0)
- moved R101 5.28 mm to (110.5, 121.0)
- moved C301 4.58 mm to (151.3, 99.1)
- moved C302 4.58 mm to (151.4, 102.4)
- moved J102 0.96 mm to (103.1, 89.5)
- renumbered C101 to C201, C102 to C202, C103 to C203, C104 to C204, C105 to C205, C106 to C206, C108 to C301, C107 to C302, J111 to J102, J102 to J201, J104 to J202, J105 to J203, J106 to J204, J108 to J205, J109 to J206, J110 to J301, R112 to R101, R113 to R102, R101 to R201, R102 to R202, R103 to R203, R104 to R204, R105 to R205, R106 to R206, R108 to R301, R109 to R302, R111 to R303, R110 to R304, R107 to R305, TP101 to TP201, TP102 to TP202, TP104 to TP203, TP106 to TP204, TP108 to TP205, TP110 to TP206, TP112 to TP207
Connections:
- J101 pad 2: Net-(A101-BAT+) -> Net-(J101-Pin_2)
Routing:
- net VDD: track 191.2 -> 222.5 mm, vias 1 -> 5
- net Net-(J101-Pin_2): track 0.00 -> 13.8 mm
- net Net-(A101-BAT-): track 22.1 -> 34.1 mm, vias 0 -> 2
- net SCL: track 36.8 -> 45.1 mm, vias 0 -> 1
- net Net-(J301-DAT1): track 3.91 -> 11.9 mm, vias 0 -> 2
- net SDA: track 55.8 -> 63.2 mm
- net Net-(J301-CLK): track 14.8 -> 20.8 mm, vias 0 -> 2
- net /SD/CLK: track 15.7 -> 10.1 mm
- net /SD/DAT0: track 36.6 -> 40.7 mm, vias 1 -> 3
- net /SD/CMD: track 39.0 -> 42.3 mm, vias 3 -> 1
- net Net-(A101-BAT+): track 25.5 -> 22.7 mm, vias 1 -> 0
- net Net-(J301-DAT3/CD): track 5.02 -> 6.46 mm, vias 0 -> 1
- net Net-(J301-DAT2): track 3.73 -> 3.99 mm, vias 0 -> 1
- net GND: vias 144 -> 171
Other:
- board text added: "OFF"
- board text added: "低温環境で使いたい場合は分圧用抵抗を47~100kΩにしてください 常温環境で分解能を高くしたい場合は10kΩにしてください 6ch同時計測可能です SDはSDMMCモードのみの対応になっています．"
- board text removed: "低温環境で使いたい場合は分圧用抵抗を100kΩにしてください 常温環境で分解能を高くしたい場合は10kΩにしてください 6ch同時計測可能です SDはSDMMCモードのみの対応になっています．"
