File: hardware/ThermistorHub/ThermistorHubSMD/Thermistor.kicad_sch (KiCad schematic)
At the start: 21 parts, among them J104 Thermistor1, J105 Thermistor2, J106 Thermistor3, J107 Thermistor4

Commit message: 途中まで
Parts:
- removed C113, C114, C115, C116: 0.1u, Capacitor_THT:C_Axial_L3.8mm_D2.6mm_P7.50mm_Horizontal, symbol Device:C
- removed R114, R116: 100k, Resistor_THT:R_Axial_DIN0204_L3.6mm_D1.6mm_P5.08mm_Horizontal, symbol Device:R
- added C501, C502, C503, C504: 100nF, Capacitor_SMD:C_0402_1005Metric, symbol Device:C
- added R506, R508: 47k, Resistor_SMD:R_0201_0603Metric, symbol Device:R
- renumbered J104 to J501, J105 to J502, J106 to J503, J107 to J504, R109 to R501, R110 to R502, R111 to R503, R112 to R504, R113 to R505, R115 to R507, TP101 to TP501, TP102 to TP502, TP103 to TP503, TP104 to TP504, TP105 to TP505
Connections:
- net AGND: now also C501.1, C502.1, C503.1, C504.1, R506.2, R508.2
- net R_Thermistor1: now also C501.2
- net R_Thermistor2: now also C502.2
- net R_Thermistor3: now also C503.2
- net R_Thermistor4: now also C504.2
- net at J504.2 (Pin_2), R507.2, TP505.1: now also R508.1
- net at J503.2 (Pin_2), R505.2, TP504.1: now also R506.1
Other:
- moved on the sheet: J501, J502, J503, J504, R501, R502, R503, R504, R505, R507, TP501, TP502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
