File: hardware/ThermistorHub/ThermistorHubSMD/Thermistor2.kicad_sch (KiCad schematic)
At the start: 20 parts, among them J108 Thermistor5, J109 Thermistor6, J110 Thermistor7, J111 Thermistor8

Commit message: 途中まで
Parts:
- removed C117, C118, C119, C120: 0.1u, Capacitor_THT:C_Axial_L3.8mm_D2.6mm_P7.50mm_Horizontal, symbol Device:C
- removed R122, R124: 100k, Resistor_THT:R_Axial_DIN0204_L3.6mm_D1.6mm_P5.08mm_Horizontal, symbol Device:R
- added C601, C602, C603, C604: 100nF, Capacitor_SMD:C_0402_1005Metric, symbol Device:C
- added R606, R608: 47k, Resistor_SMD:R_0201_0603Metric, symbol Device:R
- renumbered J108 to J601, J109 to J602, J110 to J603, J111 to J604, R117 to R601, R118 to R602, R119 to R603, R120 to R604, R121 to R605, R123 to R607, TP106 to TP601, TP107 to TP602, TP108 to TP603, TP109 to TP604
Connections:
- net AGND: now also C602.1, C603.1, C604.1, R606.2, R608.2
- net R_Thermistor5: now also C601.2
- net R_Thermistor6: now also C602.2
- net R_Thermistor7: now also C603.2
- net R_Thermistor8: now also C604.2
- net at J604.2 (Pin_2), R607.2, TP604.1: now also R608.1
- net at J603.2 (Pin_2), R605.2, TP603.1: now also R606.1
Other:
- moved on the sheet: J601, J602, J603, J604, R601, R602, R603, R604, R605, R607, TP601, TP602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
