File: hardware/ThermistorHub/ThermistorHubSMD/ThermistorADC.kicad_sch (KiCad schematic)
At the start: 10 parts, among them U102 ADS1115IRUGT, U103 ADS1115IRUGT, U104 NJM2884U1-33-TE1

Commit message: 途中まで
Parts:
- NT401: renamed from NT101; footprint (none) -> NetTie:NetTie-2_SMD_Pad2.0mm
- U401: renamed from U102; footprint ADS1115IRUGT:IC_ADS1115IRUGT -> Package_SO:VSSOP-10_3x3mm_P0.5mm
- U402: renamed from U103; footprint ADS1115IRUGT:IC_ADS1115IRUGT -> Package_SO:VSSOP-10_3x3mm_P0.5mm
- U403: renamed from U104; footprint SOT89-5-1/2_NWJ -> Library:SOT89-5-1&slash_2_NWJ
- renumbered C107 to C401, C108 to C402, C109 to C403, C110 to C404, C111 to C405, C112 to C406
Connections:
- net Thermisotr1/R_Thermistor1 renamed THR1
- net Thermisotr1/R_Thermistor2 renamed THR2
- net Thermisotr1/R_Thermistor3 renamed THR3
- net Thermisotr1/R_Thermistor4 renamed THR4
- net Thermisotr2/R_Thermistor1 renamed THR5
- net Thermisotr2/R_Thermistor2 renamed THR6
- net Thermisotr2/R_Thermistor3 renamed THR7
- net Thermisotr2/R_Thermistor4 renamed THR8
Other:
- sheet Thermisotr2 ports: added R_Thermistor5, R_Thermistor6, R_Thermistor7, R_Thermistor8; removed R_Thermistor1, R_Thermistor2, R_Thermistor3, R_Thermistor4
Changed lines of the file:
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@@
+		)
+	)
+	(label "THR5"
+		(at 82.55 129.54 0)
+		(effects
+			(font
+				(size 1.27 1.27)
+			)
+			(justify left bottom)
+		)
+	)
+	(label "THR1"
+		(at 82.55 71.12 0)
+		(effects
+			(font
+				(size 1.27 1.27)
+			)
+			(justify left bottom)
+		)
+	)
+	(label "THR7"
+		(at 82.55 134.62 0)
+		(effects
+			(font
+				(size 1.27 1.27)
+			)
+			(justify left bottom)
+		)
+	)
+	(label "THR3"
+		(at 82.55 76.2 0)
+		(effects
+			(font
+				(size 1.27 1.27)
+			)
+			(justify left bottom)
+		)
+	)
+	(label "THR8"
+		(at 82.55 137.16 0)
+		(effects
+			(font
+				(size 1.27 1.27)
+			)
+			(justify left bottom)
+		)
+	)
+	(label "THR4"
+		(at 82.55 78.74 0)
+		(effects
+			(font
+				(size 1.27 1.27)
+			)
+			(justify left bottom)
+		)
+	)
+	(label "THR6"
+		(at 82.55 132.08 0)
+		(effects
+			(font
+				(size 1.27 1.27)
+			)
+			(justify left bottom)
+		)
+	)
+	(label "THR2"
+		(at 82.55 73.66 0)
+		(effects
+			(font
+				(size 1.27 1.27)
+			)
+			(justify left bottom)
 		)
 	)
@@
 		(in_pos_files yes)
 		(dnp no)
-		(property "Reference" "C108"
+		(property "Reference" "C402"
 			(at 151.13 128.778 0)
 			(show_name no)
@@
 			(project "ThermistorHub"
 				(path "/654b68be-bf39-4999-b2d7-5e3864aa249f/0b7ca361-a991-4a4c-856d-2332484faac6"
-					(reference "C108")
+					(reference "C402")
 					(unit 1)
 				)
@@
 		(dnp no)
 		(fields_autoplaced yes)
-		(property "Reference" "U103"
+		(property "Reference" "U402"
 			(at 127 114.3 0)
 			(show_name no)
@@
 			)
 		)
-		(property "Footprint" "ADS1115IRUGT:IC_ADS1115IRUGT"
+		(property "Footprint" "Package_SO:VSSOP-10_3x3mm_P0.5mm"
 			(at 127 134.62 0)
 			(hide yes)
@@
 			(project "ThermistorHub"
 				(path "/654b68be-bf39-4999-b2d7-5e3864aa249f/0b7ca361-a991-4a4c-856d-2332484faac6"
-					(reference "U103")
+					(reference "U402")
 					(unit 1)
 				)
@@
 		(dnp no)
 		(fields_autoplaced yes)
-		(property "Reference" "NT101"
+		(property "Reference" "NT401"
 			(at 193.04 129.54 0)
 			(show_name no)
@@
 			)
 		)
-		(property "Footprint" ""
+		(property "Footprint" "NetTie:NetTie-2_SMD_Pad2.0mm"
 			(at 193.04 134.62 0)
 			(hide yes)
@@
 			(project "ThermistorHub"
 				(path "/654b68be-bf39-4999-b2d7-5e3864aa249f/0b7ca361-a991-4a4c-856d-2332484faac6"
-					(reference "NT101")
+					(reference "NT401")
 					(unit 1)
 				)
@@
 		(dnp no)
 		(fields_autoplaced yes)
-		(property "Reference" "U102"
+		(property "Reference" "U401"
 			(at 127 55.88 0)
 			(show_name no)
@@
 			)
 		)
-		(property "Footprint" "ADS1115IRUGT:IC_ADS1115IRUGT"
+		(property "Footprint" "Package_SO:VSSOP-10_3x3mm_P0.5mm"
 			(at 127 76.2 0)
 			(hide yes)
@@
 			(project "ThermistorHub"
 				(path "/654b68be-bf39-4999-b2d7-5e3864aa249f/0b7ca361-a991-4a4c-856d-2332484faac6"
-					(reference "U102")
+					(reference "U401")
 					(unit 1)
 				)
@@
 		(in_pos_files yes)
 		(dnp no)
-		(property "Reference" "C109"
+		(property "Reference" "C403"
 			(at 160.528 68.834 0)
 			(show_name no)
@@
 			(project "ThermistorHub"
 				(path "/654b68be-bf39-4999-b2d7-5e3864aa249f/0b7ca361-a991-4a4c-856d-2332484faac6"
-					(reference "C109")
+					(reference "C403")
 					(unit 1)
 				)
@@
 		(in_pos_files yes)
 		(dnp no)
-		(property "Reference" "C112"
+		(property "Reference" "C406"
 			(at 258.318 98.044 0)
 			(show_name no)
@@
 			(project "ThermistorHub"
 				(path "/654b68be-bf39-4999-b2d7-5e3864aa249f/0b7ca361-a991-4a4c-856d-2332484faac6"
-					(reference "C112")
+					(reference "C406")
 					(unit 1)
 				)
@@
 		(in_pos_files yes)
 		(dnp no)
-		(property "Reference" "C110"
+		(property "Reference" "C404"
 			(at 160.528 128.524 0)
 			(show_name no)
@@
 			(project "ThermistorHub"
 				(path "/654b68be-bf39-4999-b2d7-5e3864aa249f/0b7ca361-a991-4a4c-856d-2332484faac6"
-					(reference "C110")
+					(reference "C404")
 					(unit 1)
 				)
@@
 		(dnp no)
 		(fields_autoplaced yes)
-		(property "Reference" "U104"
+		(property "Reference" "U403"
 			(at 213.36 82.55 0)
 			(show_name no)
@@
 			)
 		)
-		(property "Footprint" "SOT89-5-1/2_NWJ"
+		(property "Footprint" "Library:SOT89-5-1&slash_2_NWJ"
 			(at 190.5 92.71 0)
 			(hide yes)
@@
 			(project "ThermistorHub"
 				(path "/654b68be-bf39-4999-b2d7-5e3864aa249f/0b7ca361-a991-4a4c-856d-2332484faac6"
-					(reference "U104")
+					(reference "U403")
 					(unit 1)
 				)
@@
 		(in_pos_files yes)
 		(dnp no)
-		(property "Reference" "C111"
+		(property "Reference" "C405"
 			(at 248.92 98.298 0)
 			(show_name no)
@@
 			(project "ThermistorHub"
 				(path "/654b68be-bf39-4999-b2d7-5e3864aa249f/0b7ca361-a991-4a4c-856d-2332484faac6"
-					(reference "C111")
+					(reference "C405")
 					(unit 1)
 				)
@@
 		(in_pos_files yes)
 		(dnp no)
-		(property "Reference" "C107"
+		(property "Reference" "C401"
 			(at 151.13 69.088 0)
 			(show_name no)
@@
 			(project "ThermistorHub"
 				(path "/654b68be-bf39-4999-b2d7-5e3864aa249f/0b7ca361-a991-4a4c-856d-2332484faac6"
-					(reference "C107")
+					(reference "C401")
 					(unit 1)
 				)
@@
 			)
 		)
-		(pin "R_Thermistor1" input
-			(at 76.2 129.54 0)
-			(effects
-				(font
-					(size 1.27 1.27)
-				)
-				(justify right)
-			)
-		)
-		(pin "R_Thermistor2" input
-			(at 76.2 132.08 0)
-			(effects
-				(font
-					(size 1.27 1.27)
-				)
-				(justify right)
-			)
-		)
-		(pin "R_Thermistor3" input
-			(at 76.2 134.62 0)
-			(effects
-				(font
-					(size 1.27 1.27)
-				)
-				(justify right)
-			)
-		)
-		(pin "R_Thermistor4" input
-			(at 76.2 137.16 0)
-			(effects
-				(font
-					(size 1.27 1.27)
-				)
-				(justify right)
-			)
-		)
 		(pin "V_Ref" input
 			(at 76.2 123.19 0)
 			(effects
 				(font
+					(size 1.27 1.27)
+				)
+				(justify right)
+			)
+		)
+		(pin "R_Thermistor5" input
+			(at 76.2 129.54 0)
+			(effects
+				(font
+					(size 1.27 1.27)
+				)
+				(justify right)
+			)
+		)
+		(pin "R_Thermistor6" input
+			(at 76.2 132.08 0)
+			(effects
+				(font
+					(size 1.27 1.27)
+				)
+				(justify right)
+			)
+		)
+		(pin "R_Thermistor7" input
+			(at 76.2 134.62 0)
+			(effects
+				(font
+					(size 1.27 1.27)
+				)
+				(justify right)
+			)
+		)
+		(pin "R_Thermistor8" input
+			(at 76.2 137.16 0)
+			(effects
+				(font
