File: hardware/ThermistorHub/ThermistorHubSMD/ThermistorHub.kicad_sch (KiCad schematic)
At the start: 6 parts, among them J101 BATPin, J102 Battery, SW101 SW_SPDT

Commit message: 途中まで
Parts:
- added D105: STAT, LED_SMD:LED_0805_2012Metric, symbol Device:LED
- added D106: ERROR, LED_SMD:LED_0805_2012Metric, symbol Device:LED
- added R108, R109, R111: 10k, Resistor_SMD:R_0402_1005Metric, symbol Device:R
- added R110, R112: 1k, Resistor_SMD:R_0402_1005Metric, symbol Device:R
- added SW501: SW_Push, symbol Switch:SW_Push
- SW101: footprint Button_Switch_THT:SW_Slide-03_Wuerth-WS-SLTV_10x2.5x6.4_P2.54mm -> Button_Switch_THT:SW_Slide_SPDT_Angled_CK_OS102011MA1Q
Connections:
- net GND: now also D105.1 (K), D106.1 (K), SW501.1
- net VDD: now also R111.1
- net at A101.1 (GPIO1): now also R110.1
- net at A101.2 (GPIO2): now also R112.1
- net SDA2: now reaches A101.4 (GPIO4)
- net SDA2: now also R108.2
- net SCL2: now reaches A101.5 (GPIO5)
- net SCL2: now also R109.2
- net at A101.6 (GPIO6): now also R111.2, SW501.2
- net SCL renamed SCL1
- net SD/CLK renamed CLK
- net SD/CMD renamed CMD
- net SD/DAT0 renamed DAT0
- net SDA renamed SDA1
- new net: D106.2 (A), R112.2
- new net: D105.2 (A), R110.2
- new net +3V0: R108.1, R109.1
- no-connect marks 4 -> 5
Other:
- added sheet BMP390 (BMP390.kicad_sch)
- added sheet Pt1000 (untitled.kicad_sch)
- added sheet TMP117 (TMP117.kicad_sch)
- note removed: "残タスク ・ThermistorのキャパシタのTHTからSMD変更 ・レギュレーターのフットプリント ・ADCのフットプリント"
