File: hardware/ThermistorHub/ThermistorHubSMD/ThermistorHub.kicad_pcb (KiCad board)
At the start: 2 copper layers, 6 parts

Commit message: 途中まで
Parts:
- removed ? (x6): , 
- added A101: ~, Library:XIAO-ESP32S3-DIP, F.Cu at (112.4, 96.3)
- added C101: 10μF, Capacitor_SMD:C_0603_1608Metric, F.Cu at (70.2, 72.0)
- added C102: 100nF, Capacitor_SMD:C_0402_1005Metric, F.Cu at (73.7, 75.4)
- added C103: 100nF, Capacitor_SMD:C_0402_1005Metric, F.Cu at (73.7, 77.4)
- added C104: 10μF, Capacitor_SMD:C_0603_1608Metric, F.Cu at (70.2, 74.5)
- added C105: 100nF, Capacitor_SMD:C_0402_1005Metric, F.Cu at (74.3, 40.0)
- added C106: 10μF, Capacitor_SMD:C_0603_1608Metric, F.Cu at (74.8, 37.8)
- added C401: 100nF, Capacitor_SMD:C_0402_1005Metric, F.Cu at (77.3, 55.2)
- added C402: 100nF, Capacitor_SMD:C_0402_1005Metric, F.Cu at (77.3, 57.2)
- added C403: 10μF, Capacitor_SMD:C_0603_1608Metric, F.Cu at (77.8, 62.5)
- added C404: 10μF, Capacitor_SMD:C_0603_1608Metric, F.Cu at (77.8, 65.0)
- added C405: 100nF, Capacitor_SMD:C_0402_1005Metric, F.Cu at (114.0, 66.0)
- added C406: 10μF, Capacitor_SMD:C_0603_1608Metric, F.Cu at (114.0, 64.0)
- added C501: 100nF, Capacitor_SMD:C_0402_1005Metric, F.Cu at (39.8, 72.0)
- added C502: 100nF, Capacitor_SMD:C_0402_1005Metric, F.Cu at (39.8, 74.0)
- added C503: 100nF, Capacitor_SMD:C_0402_1005Metric, F.Cu at (39.8, 76.0)
- added C504: 100nF, Capacitor_SMD:C_0402_1005Metric, F.Cu at (39.8, 77.9)
- added C601: 100nF, Capacitor_SMD:C_0402_1005Metric, F.Cu at (64.8, 55.2)
- added C602: 100nF, Capacitor_SMD:C_0402_1005Metric, F.Cu at (64.8, 57.2)
- added C603: 100nF, Capacitor_SMD:C_0402_1005Metric, F.Cu at (64.8, 59.2)
- added C604: 100nF, Capacitor_SMD:C_0402_1005Metric, F.Cu at (64.8, 61.1)
- added J101: BATPin, Connector_JST:JST_PH_B2B-PH-K_1x02_P2.00mm_Vertical, F.Cu at (126.0, 95.5)
- added J102: Battery, Connector_JST:JST_PH_B2B-PH-K_1x02_P2.00mm_Vertical, F.Cu at (126.0, 102.0)
- added J301: Micro_SD_Card_Det_Hirose_DM3AT, Connector_Card:microSD_HC_Hirose_DM3AT-SF-PEJM5, F.Cu at (148.0, 96.5)
- added J501: Thermistor1, Connector_JST:JST_PH_B2B-PH-K_1x02_P2.00mm_Vertical, F.Cu at (107.0, 127.0)
- added J502: Thermistor2, Connector_JST:JST_PH_B2B-PH-K_1x02_P2.00mm_Vertical, F.Cu at (121.0, 127.0)
- added J503: Thermistor3, Connector_JST:JST_PH_B2B-PH-K_1x02_P2.00mm_Vertical, F.Cu at (135.0, 127.0)
- added J504: Thermistor4, Connector_JST:JST_PH_B2B-PH-K_1x02_P2.00mm_Vertical, F.Cu at (149.0, 127.0)
- added J601: Thermistor5, Connector_JST:JST_PH_B2B-PH-K_1x02_P2.00mm_Vertical, F.Cu at (107.0, 118.0)
- added J602: Thermistor6, Connector_JST:JST_PH_B2B-PH-K_1x02_P2.00mm_Vertical, F.Cu at (121.0, 118.0)
- added J603: Thermistor7, Connector_JST:JST_PH_B2B-PH-K_1x02_P2.00mm_Vertical, F.Cu at (135.0, 118.0)
- added J604: Thermistor8, Connector_JST:JST_PH_B2B-PH-K_1x02_P2.00mm_Vertical, F.Cu at (149.0, 118.0)
- added NT401: NetTie_2, NetTie:NetTie-2_SMD_Pad2.0mm, F.Cu at (98.0, 52.0)
- added R101: 10k, Resistor_SMD:R_0402_1005Metric, F.Cu at (38.8, 49.2)
- added R102: 10k, Resistor_SMD:R_0402_1005Metric, F.Cu at (38.8, 51.2)
- added R103: 10k, Resistor_SMD:R_0402_1005Metric, F.Cu at (74.3, 25.6)
- added R104: 10k, Resistor_SMD:R_0402_1005Metric, F.Cu at (74.3, 27.6)
- added R105: 10k, Resistor_SMD:R_0402_1005Metric, F.Cu at (74.3, 29.6)
- added R106: 10k, Resistor_SMD:R_0402_1005Metric, F.Cu at (74.3, 31.6)
- added R107: 10k, Resistor_SMD:R_0402_1005Metric, F.Cu at (74.3, 33.6)
- added R303: 33Ω, Resistor_SMD:R_0402_1005Metric, F.Cu at (74.3, 35.5)
- added R501: 1k, Resistor_SMD:R_0201_0603Metric, F.Cu at (39.6, 55.1)
- added R502: 47k, Resistor_SMD:R_0201_0603Metric, F.Cu at (39.6, 56.9)
- added R503: 1k, Resistor_SMD:R_0201_0603Metric, F.Cu at (39.6, 58.6)
- added R504: 47k, Resistor_SMD:R_0201_0603Metric, F.Cu at (39.6, 60.4)
- added R505: 1k, Resistor_SMD:R_0201_0603Metric, F.Cu at (39.6, 62.1)
- added R506: 47k, Resistor_SMD:R_0201_0603Metric, F.Cu at (39.9, 66.5)
- added R507: 1k, Resistor_SMD:R_0201_0603Metric, F.Cu at (39.6, 63.9)
- added R508: 47k, Resistor_SMD:R_0201_0603Metric, F.Cu at (39.9, 68.2)
- added R601: 1k, Resistor_SMD:R_0201_0603Metric, F.Cu at (62.1, 55.1)
- added R602: 47k, Resistor_SMD:R_0201_0603Metric, F.Cu at (62.1, 56.9)
- added R603: 1k, Resistor_SMD:R_0201_0603Metric, F.Cu at (62.1, 58.6)
- added R604: 47k, Resistor_SMD:R_0201_0603Metric, F.Cu at (62.1, 60.4)
- added R605: 1k, Resistor_SMD:R_0201_0603Metric, F.Cu at (62.1, 62.1)
- added R606: 47k, Resistor_SMD:R_0201_0603Metric, F.Cu at (64.5, 67.8)
- added R607: 1k, Resistor_SMD:R_0201_0603Metric, F.Cu at (62.1, 63.9)
- added R608: 47k, Resistor_SMD:R_0201_0603Metric, F.Cu at (64.5, 69.6)
- added SW101: SW_SPDT, Button_Switch_THT:SW_Slide_SPDT_Angled_CK_OS102011MA1Q, F.Cu at (132.0, 88.0)
- added TP501: TestPoint, Connector_PinHeader_2.54mm:PinHeader_1x01_P2.54mm_Vertical, F.Cu at (102.0, 118.0)
- added TP502: TestPoint, Connector_PinHeader_2.54mm:PinHeader_1x01_P2.54mm_Vertical, F.Cu at (114.0, 127.0)
- added TP503: TestPoint, Connector_PinHeader_2.54mm:PinHeader_1x01_P2.54mm_Vertical, F.Cu at (128.0, 127.0)
- added TP504: TestPoint, Connector_PinHeader_2.54mm:PinHeader_1x01_P2.54mm_Vertical, F.Cu at (142.0, 127.0)
- added TP505: TestPoint, Connector_PinHeader_2.54mm:PinHeader_1x01_P2.54mm_Vertical, F.Cu at (156.0, 127.0)
- added TP601: TestPoint, Connector_PinHeader_2.54mm:PinHeader_1x01_P2.54mm_Vertical, F.Cu at (114.0, 118.0)
- added TP602: TestPoint, Connector_PinHeader_2.54mm:PinHeader_1x01_P2.54mm_Vertical, F.Cu at (128.0, 118.0)
- added TP603: TestPoint, Connector_PinHeader_2.54mm:PinHeader_1x01_P2.54mm_Vertical, F.Cu at (142.0, 118.0)
- added TP604: TestPoint, Connector_PinHeader_2.54mm:PinHeader_1x01_P2.54mm_Vertical, F.Cu at (156.0, 118.0)
- added U101: ~, WOBCLibrary:BME280, F.Cu at (135.0, 96.0)
- added U401: ADS1115IRUGT, Package_SO:VSSOP-10_3x3mm_P0.5mm, F.Cu at (117.0, 111.0)
- added U402: ADS1115IRUGT, Package_SO:VSSOP-10_3x3mm_P0.5mm, F.Cu at (109.2, 111.0)
- added U403: NJM2884U1-33-TE1, Library:SOT89-5-1&slash_2_NWJ, F.Cu at (111.5, 70.0)
Other:
- copper layers 2 -> 4

Commit message: おいた
Parts:
- removed TP501, TP502, TP503, TP504, TP505, TP601, TP602, TP603, TP604: TestPoint, Connector_PinHeader_2.54mm:PinHeader_1x01_P2.54mm_Vertical
- added B501: ~, WOBCLibrary:Board_1U_60x60, F.Cu at (159.1, 101.9)
- added C107: 10μF, Capacitor_SMD:C_0603_1608Metric, F.Cu at (180.6, 107.2)
- added C108: 100nF, Capacitor_SMD:C_0402_1005Metric, F.Cu at (180.1, 106.0)
- added C109: 10μF, Capacitor_SMD:C_0603_1608Metric, F.Cu at (176.7, 103.5)
- added C110: 100nF, Capacitor_SMD:C_0402_1005Metric, F.Cu at (175.5, 104.7)
- added C407: 100nF, Capacitor_SMD:C_0402_1005Metric, F.Cu at (180.8, 113.6)
- added C408: 10μF, Capacitor_SMD:C_0603_1608Metric, F.Cu at (181.4, 114.9)
- added D105: STAT, LED_SMD:LED_0805_2012Metric, F.Cu at (136.8, 86.3)
- added D106: ERROR, LED_SMD:LED_0805_2012Metric, F.Cu at (136.8, 90.2)
- added R108: 10k, Resistor_SMD:R_0402_1005Metric, F.Cu at (137.0, 104.0)
- added R109: 10k, Resistor_SMD:R_0402_1005Metric, F.Cu at (137.0, 105.1)
- added R110: 1k, Resistor_SMD:R_0402_1005Metric, F.Cu at (139.1, 86.1)
- added R111: 10k, Resistor_SMD:R_0402_1005Metric, F.Cu at (137.6, 94.0)
- added R112: 1k, Resistor_SMD:R_0402_1005Metric, F.Cu at (139.1, 88.3)
- added SW501: SW_Push, WOBCLibrary:TVAF06-A020B-R, F.Cu at (137.0, 97.6)
- added U501: BMP390, Library:10LGA_2X2X0p75_BOS, F.Cu at (177.8, 105.4)
- added U502: TMP117xxDRV, Package_SON:WSON-6-1EP_2x2mm_P0.65mm_EP1x1.6mm, F.Cu at (178.5, 114.0)
- R501, R503, R505, R507, R601, R603, R605, R607: footprint Resistor_SMD:R_0201_0603Metric -> Resistor_SMD:R_0402_1005Metric
- R502, R504, R506, R508, R602, R604, R606, R608: footprint Resistor_SMD:R_0201_0603Metric -> Resistor_SMD:R_0603_1608Metric
- moved R502 147.7 mm to (173.9, 118.2)
- moved R504 139.7 mm to (166.7, 118.2)
- moved R102 138.3 mm to (167.3, 102.3), turned to 90 degrees
- moved R101 138.1 mm to (166.3, 102.3), turned to 90 degrees
- moved R506 130.5 mm to (159.7, 118.2)
- moved R501 125.4 mm to (145.6, 122.1)
- moved R602 123.5 mm to (173.6, 110.1)
- moved R508 123.1 mm to (152.4, 118.2)
- moved R503 122.6 mm to (145.6, 120.1)
- moved R505 118.7 mm to (145.6, 115.5)
- moved R507 117.1 mm to (145.6, 113.6)
- moved C502 115.8 mm to (145.6, 121.1), turned to 180 degrees
- moved R604 115.8 mm to (166.7, 110.1)
- moved C501 115.1 mm to (143.7, 121.5)
- moved R104 114.3 mm to (165.5, 96.4)
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Connections:
- net /SD/CLK renamed /CLK
- net /SD/CMD renamed /CMD
- net /SD/DAT0 renamed /DAT0
- net /Thermistor/Thermisotr1/R_Thermistor1 renamed /Thermistor/THR1
- net /Thermistor/Thermisotr1/R_Thermistor2 renamed /Thermistor/THR2
- net /Thermistor/Thermisotr1/R_Thermistor3 renamed /Thermistor/THR3
- net /Thermistor/Thermisotr1/R_Thermistor4 renamed /Thermistor/THR4
- net /Thermistor/Thermisotr2/R_Thermistor5 renamed /Thermistor/THR5
- net /Thermistor/Thermisotr2/R_Thermistor6 renamed /Thermistor/THR6
- net /Thermistor/Thermisotr2/R_Thermistor7 renamed /Thermistor/THR7
- net /Thermistor/Thermisotr2/R_Thermistor8 renamed /Thermistor/THR8
- A101 pad 1: unconnected-(A101-GPIO1-Pad1) -> Net-(A101-GPIO1)
- A101 pad 2: unconnected-(A101-GPIO2-Pad2) -> Net-(A101-GPIO2)
- A101 pad 4: unconnected-(A101-GPIO4-Pad4) -> SDA2
- A101 pad 5: unconnected-(A101-GPIO5-Pad5) -> SCL2
- A101 pad 6: unconnected-(A101-GPIO6-Pad6) -> Net-(A101-GPIO6)
- A101 pad 7: SCL -> SCL1
- A101 pad 8: SDA -> SDA1
- C601 pad 1: unconnected-(C601-Pad1) -> /Thermistor/Thermisotr2/AGND
- R101 pad 2: SDA -> SDA1
- R102 pad 2: SCL -> SCL1
- U101 pad 3: SDA -> SDA1
- U101 pad 4: SCL -> SCL1
- U401 pad 10: SCL -> SCL2
- U401 pad 9: SDA -> SDA2
- U402 pad 10: SCL -> SCL2
- U402 pad 9: SDA -> SDA2
Other:
- board outline added: 50 x 50 mm
